File: QMS.kicad_pcb (KiCad board)
At the start: 2 copper layers, 58.4 x 63.5 mm, 12 parts, among them J1 Screw_Terminal_01x02, J2 PINHD_1x5_Male, J3 PINHD_1x3_Male, U1 ESP-12E, U2 AMS1117-3.3

Commit message: updated accordin to suggested rules
Parts:
- removed C1, C2: C_Polarized_US, Capacitor_THT:CP_Radial_D6.3mm_P2.50mm
- removed J1: Screw_Terminal_01x02, TerminalBlock:TerminalBlock_MaiXu_MX126-5.0-02P_1x02_P5.00mm
- removed J2: PINHD_1x5_Male, Connector_PinHeader_2.54mm:PinHeader_1x05_P2.54mm_Vertical
- removed J3: PINHD_1x3_Male, Connector_PinHeader_2.54mm:PinHeader_1x03_P2.54mm_Vertical
- removed P1, P2: ~, Button_Switch_THT:SW_PUSH-12mm
- removed R1, R2: Resistor, Resistor_THT:R_Axial_DIN0207_L6.3mm_D2.5mm_P7.62mm_Horizontal
- removed U1: ESP-12E, RF_Module:ESP-12E
- removed U2: AMS1117-3.3, Package_TO_SOT_SMD:SOT-223-3_TabPin2
- removed U3: ~, MyConnectors:Hub16
- added C3: C_Polarized_US, MyConnectors:CP_Radial_D6.3mm_P2.50mm, F.Cu at (127.0, 111.8)
- added C4: C_Polarized_US, MyConnectors:CP_Radial_D6.3mm_P2.50mm, F.Cu at (127.0, 101.6)
- added J4: Conn_02x08_Top_Bottom, MyConnectors:PinHeader 2x8 p2.54mm, F.Cu at (144.8, 71.1)
- added J6: Screw_Terminal_01x02, TerminalBlock:TerminalBlock_MaiXu_MX126-5.0-02P_1x02_P5.00mm, F.Cu at (129.6, 121.9)
- added J7: PINHD_1x5_Male, MyConnectors:PinHeader_1x05_P2.54mm_Vertical, F.Cu at (139.7, 99.1)
- added J8: PINHD_1x5_Male, MyConnectors:PinHeader_1x05_P2.54mm_Vertical, F.Cu at (147.3, 99.1)
- added P3: ~, MyConnectors:PUSH_BTN_12x12mm, F.Cu at (101.2, 73.7)
- added P4: ~, MyConnectors:PUSH_BTN_12x12mm, F.Cu at (101.2, 116.9)
- added R3: Resistor, MyConnectors:R_Axial_DIN0207_L6.3mm_D2.5mm_P7.62mm_Horizontal, F.Cu at (101.6, 91.4)
- added R4: Resistor, MyConnectors:R_Axial_DIN0207_L6.3mm_D2.5mm_P7.62mm_Horizontal, F.Cu at (101.6, 99.1)
- added U4: ESP-12E, RF_Module:ESP-12E, F.Cu at (127.0, 79.7)
- added U5: AMS1117-3.3, Package_TO_SOT_SMD:SOT-223-3_TabPin2, F.Cu at (145.4, 121.9)
Routing:
- net Net-(U1-VCC): track 160.0 -> 0.00 mm
- net /VCC: track 0.00 -> 155.6 mm
- net GND: track 230.4 -> 113.3 mm
- net /GPIO5: track 0.00 -> 104.2 mm, vias 0 -> 1
- net Net-(U1-GPIO5): track 97.1 -> 0.00 mm, vias 1 -> 0
- net /GPIO3/RXD: track 0.00 -> 88.4 mm, vias 0 -> 1
- net /RST: track 0.00 -> 74.0 mm, vias 0 -> 1
- net /EN: track 0.00 -> 70.6 mm, vias 0 -> 1
- net Net-(U1-GPIO0): track 68.4 -> 0.00 mm, vias 1 -> 0
- net /GPIO14: track 0.00 -> 62.9 mm, vias 0 -> 1
- net Net-(U1-GPIO15): track 60.3 -> 0.00 mm, vias 1 -> 0
- net /GPIO4: track 0.00 -> 57.7 mm, vias 0 -> 1
- net /GPIO0: track 0.00 -> 56.5 mm, vias 0 -> 1
- net /GPIO15: track 0.00 -> 54.1 mm, vias 0 -> 1
- net Net-(U1-GPIO13): track 53.2 -> 0.00 mm, vias 2 -> 0
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
Commit message: some small fixes
Connections:
- U4 pad 17: /GPIO2 -> /VCC
Routing:
- net /VCC: track 155.6 -> 231.2 mm, vias 0 -> 2
- net /GPIO5: track 104.2 -> 96.1 mm
- net /RST: track 74.0 -> 67.1 mm
- net /GPIO0: track 56.5 -> 52.1 mm

Commit message: added changes
Parts:
- J8: footprint MyConnectors:PinHeader_1x05_P2.54mm_Vertical -> Connector_PinHeader_2.54mm:PinHeader_1x02_P2.54mm_Vertical
- moved J8 2.54 mm to (149.9, 99.1)
Connections:
- J8 pad 1: /GPIO0 -> GND
- J8 pad 2: /GPIO15 -> /GPIO0
- U4 pad 16: /GPIO15 -> GND
Routing:
- net /VCC: track 231.2 -> 145.1 mm, vias 2 -> 0
- net /EN: track 70.6 -> 0.00 mm, vias 1 -> 0
- net /GPIO15: track 54.1 -> 0.00 mm, vias 1 -> 0
- net /GPIO3/RXD: track 88.4 -> 35.7 mm, vias 1 -> 0
- net /GPIO5: track 96.1 -> 65.4 mm
- net /GPIO1/TXD: track 35.3 -> 46.6 mm
- net GND: track 113.3 -> 105.4 mm
- net /RST: track 67.1 -> 59.8 mm
- net /GPIO14: track 62.9 -> 57.0 mm
- net /GPIO16: track 39.7 -> 34.0 mm
- net /GPIO12: track 45.1 -> 50.8 mm
- net /GPIO13: track 47.2 -> 41.6 mm
- net /GPIO4: track 57.3 -> 62.5 mm
- net /GPIO0: track 52.1 -> 56.6 mm
