File: QMS.kicad_pcb (KiCad board)
At the start: 2 copper layers, 58.4 x 63.5 mm, 12 parts, among them J4 Conn_02x08_Top_Bottom, J6 Screw_Terminal_01x02, J7 PINHD_1x5_Male, J8 PINHD_1x5_Male, U4 ESP-12E, U5 AMS1117-3.3

Commit message: fixed all errors
Parts:
- U4, U5: moved to B.Cu
- moved J8 27.3 mm to (133.8, 121.2)
- moved U5 22.0 mm to (123.4, 121.8), turned to 180 degrees
- moved J6 13.6 mm to (143.2, 121.2)
- moved J7 9.99 mm to (149.7, 98.1)
- moved C4 8.20 mm to (134.2, 105.5)
- moved C3 7.69 mm to (122.5, 105.5)
- moved U4 3.56 mm to (129.7, 82.0), turned to 180 degrees
- moved J4 2.59 mm to (147.3, 71.5)
- moved R3 2.55 mm to (103.2, 93.5)
- moved R4 2.55 mm to (103.2, 101.1)
- moved P4 1.30 mm to (101.2, 115.6)
- moved P3 0.86 mm to (101.2, 74.6)
Connections:
- U4 pad 3: /EN -> /VCC
Routing:
- net /GPIO0: track 56.6 -> 99.2 mm
- net /GPIO14: track 57.0 -> 28.3 mm, vias 1 -> 0
- net GND: track 105.4 -> 130.2 mm
- net /RST: track 59.8 -> 36.9 mm
- net /GPIO1/TXD: track 46.6 -> 66.9 mm, vias 0 -> 1
- net Net-(J6-Pin_1): track 24.8 -> 41.3 mm
- net /GPIO13: track 41.6 -> 25.1 mm
- net /GPIO12: track 50.8 -> 35.1 mm, vias 1 -> 0
- net /GPIO5: track 65.4 -> 53.0 mm
- net /GPIO4: track 62.5 -> 51.2 mm, vias 1 -> 0
- net /VCC: track 145.1 -> 155.7 mm
- net /GPIO16: track 34.0 -> 23.8 mm, vias 1 -> 0
- net /GPIO3/RXD: track 35.7 -> 40.4 mm, vias 0 -> 1

Commit message: marked as final
Parts:
- renumbered J8 to J1
