File: QMS.kicad_sch (KiCad schematic)
At the start: 4 parts, among them J1 Screw_Terminal_01x02, U1 ESP-12E, U2 AMS1117-3.3

Commit message: least
Parts:
- added J2: PINHD_1x5_Male, Connector_PinHeader_2.54mm:PinHeader_1x05_P2.54mm_Vertical, symbol PCM_SL_Pin_Headers:PINHD_1x5_Male
Connections:
- net GND: now also J2.1
- net at U1.1 (~{RST}): now also J2.3
- net at U1.21 (GPIO3/RXD): now also J2.5
- net at U1.22 (GPIO1/TXD): now also J2.4
- net at U1.8 (VCC), U2.2 (VO): now also J2.2

Commit message: complete
Parts:
- added J3: PINHD_1x3_Male, Connector_PinHeader_2.54mm:PinHeader_1x03_P2.54mm_Vertical, symbol PCM_SL_Pin_Headers:PINHD_1x3_Male
Connections:
- net GND: now also J3.3
- net at U1.16 (GPIO15), U3.1 (Pin_1): now also J3.2
- net at U1.18 (GPIO0), U3.13 (Pin_13): now also J3.1
Other:
- moved on the sheet: J1, J2, U1, U2

Commit message: complete
Connections:
- net GND: now also J1.1 (Pin_1); no longer J1.2 (Pin_2)
- net VCC 3.3v: now reaches J2.2, U1.8 (VCC), U2.2 (VO)
- net RESET: now reaches J2.3, U1.1 (~{RST})
- net TX: now reaches J2.4, U1.22 (GPIO1/TXD)
- net RX: now reaches J2.5, U1.21 (GPIO3/RXD)
- net at U2.3 (VI): now also J1.2 (Pin_2); no longer J1.1 (Pin_1)
Changed lines of the file:
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@@
-	(wire
-		(pts
-			(xy 100.33 95.25) (xy 100.33 119.38)
-		)
-		(stroke
-			(width 0)
-			(type default)
-		)
-	)
 	(wire
 		(pts
@@
 	(wire
 		(pts
+			(xy 100.33 92.71) (xy 106.68 92.71)
+		)
+		(stroke
+			(width 0)
+			(type default)
+		)
+	)
+	(wire
+		(pts
 			(xy 123.19 67.31) (xy 130.81 67.31)
 		)
@@
 	(wire
 		(pts
+			(xy 119.38 59.69) (xy 130.81 59.69)
+		)
+		(stroke
+			(width 0)
+			(type default)
+		)
+	)
+	(wire
+		(pts
+			(xy 190.5 107.95) (xy 213.36 107.95)
+		)
+		(stroke
+			(width 0)
+			(type default)
+		)
+	)
+	(wire
+		(pts
+			(xy 157.48 125.73) (xy 157.48 138.43)
+		)
+		(stroke
+			(width 0)
+			(type default)
+		)
+	)
+	(wire
+		(pts
+			(xy 158.75 135.89) (xy 162.56 135.89)
+		)
+		(stroke
+			(width 0)
+			(type default)
+		)
+	)
+	(wire
+		(pts
+			(xy 120.65 87.63) (xy 120.65 107.95)
+		)
+		(stroke
+			(width 0)
+			(type default)
+		)
+	)
+	(wire
+		(pts
+			(xy 156.21 92.71) (xy 156.21 107.95)
+		)
+		(stroke
+			(width 0)
+			(type default)
+		)
+	)
+	(wire
+		(pts
+			(xy 205.74 121.92) (xy 156.21 121.92)
+		)
+		(stroke
+			(width 0)
+			(type default)
+		)
+	)
+	(wire
+		(pts
+			(xy 100.33 92.71) (xy 100.33 119.38)
+		)
+		(stroke
+			(width 0)
+			(type default)
+		)
+	)
+	(wire
+		(pts
+			(xy 167.64 113.03) (xy 152.4 113.03)
+		)
+		(stroke
+			(width 0)
+			(type default)
+		)
+	)
+	(wire
+		(pts
+			(xy 213.36 123.19) (xy 167.64 123.19)
+		)
+		(stroke
+			(width 0)
+			(type default)
+		)
+	)
+	(wire
+		(pts
+			(xy 157.48 138.43) (xy 162.56 138.43)
+		)
+		(stroke
+			(width 0)
+			(type default)
+		)
+	)
+	(wire
+		(pts
+			(xy 158.75 128.27) (xy 158.75 135.89)
+		)
+		(stroke
+			(width 0)
+			(type default)
+		)
+	)
+	(wire
+		(pts
 			(xy 120.65 62.23) (xy 120.65 87.63)
 		)
@@
 	(wire
 		(pts
-			(xy 119.38 59.69) (xy 130.81 59.69)
-		)
-		(stroke
-			(width 0)
-			(type default)
-		)
-	)
-	(wire
-		(pts
-			(xy 190.5 107.95) (xy 213.36 107.95)
-		)
-		(stroke
-			(width 0)
-			(type default)
-		)
-	)
-	(wire
-		(pts
-			(xy 157.48 125.73) (xy 157.48 138.43)
-		)
-		(stroke
-			(width 0)
-			(type default)
-		)
-	)
-	(wire
-		(pts
-			(xy 158.75 135.89) (xy 162.56 135.89)
-		)
-		(stroke
-			(width 0)
-			(type default)
-		)
-	)
-	(wire
-		(pts
-			(xy 120.65 87.63) (xy 120.65 107.95)
-		)
-		(stroke
-			(width 0)
-			(type default)
-		)
-	)
-	(wire
-		(pts
-			(xy 156.21 92.71) (xy 156.21 107.95)
-		)
-		(stroke
-			(width 0)
-			(type default)
-		)
-	)
-	(wire
-		(pts
-			(xy 205.74 121.92) (xy 156.21 121.92)
-		)
-		(stroke
-			(width 0)
-			(type default)
-		)
-	)
-	(wire
-		(pts
-			(xy 167.64 113.03) (xy 152.4 113.03)
-		)
-		(stroke
-			(width 0)
-			(type default)
-		)
-	)
-	(wire
-		(pts
-			(xy 213.36 123.19) (xy 167.64 123.19)
-		)
-		(stroke
-			(width 0)
-			(type default)
-		)
-	)
-	(wire
-		(pts
-			(xy 157.48 138.43) (xy 162.56 138.43)
-		)
-		(stroke
-			(width 0)
-			(type default)
-		)
-	)
-	(wire
-		(pts
-			(xy 158.75 128.27) (xy 158.75 135.89)
-		)
-		(stroke
-			(width 0)
-			(type default)
-		)
-	)
-	(wire
-		(pts
 			(xy 190.5 97.79) (xy 205.74 97.79)
 		)
@@
 	(wire
 		(pts
-			(xy 102.87 92.71) (xy 102.87 107.95)
-		)
-		(stroke
-			(width 0)
-			(type default)
-		)
-	)
-	(wire
-		(pts
 			(xy 190.5 110.49) (xy 220.98 110.49)
 		)
@@
 	(wire
 		(pts
+			(xy 102.87 95.25) (xy 102.87 107.95)
+		)
+		(stroke
+			(width 0)
+			(type default)
+		)
+	)
+	(wire
+		(pts
 			(xy 167.64 123.19) (xy 167.64 113.03)
 		)
@@
 	(wire
 		(pts
+			(xy 124.46 69.85) (xy 130.81 69.85)
+		)
+		(stroke
+			(width 0)
+			(type default)
+		)
+	)
+	(wire
+		(pts
 			(xy 187.96 100.33) (xy 160.02 100.33)
 		)
@@
 	(wire
 		(pts
-			(xy 106.68 95.25) (xy 100.33 95.25)
-		)
-		(stroke
-			(width 0)
-			(type default)
-		)
-	)
-	(wire
-		(pts
 			(xy 156.21 118.11) (xy 152.4 118.11)
 		)
@@
 	(wire
 		(pts
-			(xy 130.81 69.85) (xy 124.46 69.85)
-		)
-		(stroke
-			(width 0)
-			(type default)
-		)
-	)
-	(wire
-		(pts
 			(xy 220.98 83.82) (xy 166.37 83.82)
 		)
@@
 	(wire
 		(pts
-			(xy 106.68 92.71) (xy 102.87 92.71)
+			(xy 102.87 95.25) (xy 106.68 95.25)
 		)
 		(stroke
@@
 			(width 0)
 			(type default)
+		)
+	)
+	(label "VCC"
+		(at 110.49 99.06 0)
+		(effects
+			(font
+				(size 1.016 1.016)
+			)
+			(justify left bottom)
+		)
+	)
+	(label "GND"
+		(at 110.49 90.17 0)
+		(effects
+			(font
+				(size 1.016 1.016)
+			)
+			(justify left bottom)
+		)
+	)
+	(label "JUMPER ONLY FOR FLASHING"
+		(at 156.21 143.51 0)
+		(effects
+			(font
+				(size 1.27 1.27)
+			)
+			(justify left bottom)
 		)
 	)
@@
 			)
 			(justify left bottom)
+		)
+	)
+	(label "RESET"
+		(at 125.73 64.77 0)
+		(effects
+			(font
+				(size 1.016 1.016)
+			)
+			(justify left bottom)
+		)
+	)
+	(label "VCC 3.3v"
+		(at 123.19 62.23 0)
+		(effects
+			(font
+				(size 1.016 1.016)
+			)
+			(justify left bottom)
+		)
+	)
+	(label "GND"
+		(at 128.27 59.69 0)
+		(effects
+			(font
+				(size 1.016 1.016)
+			)
+			(justify left bottom)
+		)
+	)
+	(label "TX"
+		(at 129.54 67.31 0)
+		(effects
+			(font
+				(size 1.016 1.016)
+			)
+			(justify left bottom)
+		)
+	)
+	(label "RX"
+		(at 129.54 69.85 0)
+		(effects
+			(font
+				(size 1.016 1.016)
+			)
+			(justify left bottom)

Commit message: completed
Parts:
- added P1, P2: ~, Button_Switch_THT:SW_PUSH-12mm, symbol PCM_Nuova-Elettronica-Switches:Push_Button
- added R1, R2: Resistor, Resistor_THT:R_Axial_DIN0207_L6.3mm_D2.5mm_P7.62mm_Horizontal, symbol PCM_SL_Resistors:Resistor
Connections:
- net GND: now also R1.1, R2.1
- net VCC 3.3v: now also P1.2, P2.1
- net at U1.19 (GPIO4): now also P1.1, R1.2
- net at U1.20 (GPIO5): now also P2.2, R2.2
