File: QMS.kicad_sch (KiCad schematic)
At the start: 12 parts, among them J1 Screw_Terminal_01x02, J2 PINHD_1x5_Male, J3 PINHD_1x3_Male, U1 ESP-12E, U2 AMS1117-3.3

Commit message: updated accordin to suggested rules
Parts:
- removed C1, C2: C_Polarized_US, Capacitor_THT:CP_Radial_D6.3mm_P2.50mm, symbol Device:C_Polarized_US
- removed J1: Screw_Terminal_01x02, TerminalBlock:TerminalBlock_MaiXu_MX126-5.0-02P_1x02_P5.00mm, symbol Connector:Screw_Terminal_01x02
- removed J2: PINHD_1x5_Male, Connector_PinHeader_2.54mm:PinHeader_1x05_P2.54mm_Vertical, symbol PCM_SL_Pin_Headers:PINHD_1x5_Male
- removed J3: PINHD_1x3_Male, Connector_PinHeader_2.54mm:PinHeader_1x03_P2.54mm_Vertical, symbol PCM_SL_Pin_Headers:PINHD_1x3_Male
- removed P1, P2: ~, Button_Switch_THT:SW_PUSH-12mm, symbol PCM_Nuova-Elettronica-Switches:Push_Button
- removed R1, R2: Resistor, Resistor_THT:R_Axial_DIN0207_L6.3mm_D2.5mm_P7.62mm_Horizontal, symbol PCM_SL_Resistors:Resistor
- removed U1: ESP-12E, RF_Module:ESP-12E, symbol RF_Module:ESP-12E
- removed U2: AMS1117-3.3, Package_TO_SOT_SMD:SOT-223-3_TabPin2, symbol Regulator_Linear:AMS1117-3.3
- removed U3: ~, MyConnectors:Hub16, symbol New_Library:HUB16
- added C3, C4: C_Polarized_US, MyConnectors:CP_Radial_D6.3mm_P2.50mm, symbol Device:C_Polarized_US
- added J4: Conn_02x08_Top_Bottom, MyConnectors:PinHeader 2x8 p2.54mm, symbol Connector_Generic:Conn_02x08_Top_Bottom
- added J6: Screw_Terminal_01x02, TerminalBlock:TerminalBlock_MaiXu_MX126-5.0-02P_1x02_P5.00mm, symbol Connector:Screw_Terminal_01x02
- added J7, J8: PINHD_1x5_Male, MyConnectors:PinHeader_1x05_P2.54mm_Vertical, symbol PCM_SL_Pin_Headers:PINHD_1x5_Male
- added P3, P4: ~, MyConnectors:PUSH_BTN_12x12mm, symbol PCM_Nuova-Elettronica-Switches:Push_Button
- added R3, R4: Resistor, MyConnectors:R_Axial_DIN0207_L6.3mm_D2.5mm_P7.62mm_Horizontal, symbol PCM_SL_Resistors:Resistor
- added U4: ESP-12E, RF_Module:ESP-12E, symbol RF_Module:ESP-12E
- added U5: AMS1117-3.3, Package_TO_SOT_SMD:SOT-223-3_TabPin2, symbol Regulator_Linear:AMS1117-3.3
Connections:
- net GND: now also C3.2, C4.2, J6.2 (Pin_2), J7.1, J8.3, R3.1, R4.1, U4.15 (GND), U5.1 (GND)
- new net: C3.1, J6.1 (Pin_1), U5.3 (VI)
- new net ADC: U4.2 (ADC)
- new net CS0: U4.9 (CS0)
- new net EN: J8.4, U4.3 (EN)
- new net GPIO0: J4.13 (Pin_13), J8.1, U4.18 (GPIO0)
- new net GPIO1/TXD: U4.22 (GPIO1/TXD)
- new net GPIO10: U4.12 (GPIO10)
- new net GPIO12: J4.10 (Pin_10), U4.6 (GPIO12)
- new net GPIO13: J4.14 (Pin_14), U4.7 (GPIO13)
- new net GPIO14: J4.12 (Pin_12), U4.5 (GPIO14)
- new net GPIO15: J4.1 (Pin_1), J8.2, U4.16 (GPIO15)
- new net GPIO16: J4.9 (Pin_9), U4.4 (GPIO16)
- new net GPIO1/TXD: J7.4
- new net GPIO2: U4.17 (GPIO2)
- new net GPIO3/RXD: U4.21 (GPIO3/RXD)
- new net GPIO3/RXD: J7.5
- new net GPIO4: P3.1, R3.2, U4.19 (GPIO4)
- new net GPIO5: P4.1, R4.2, U4.20 (GPIO5)
- new net GPIO9: U4.11 (GPIO9)
- new net MISO: U4.10 (MISO)
- new net MOSI: U4.13 (MOSI)
- new net Pin_2: J4.2 (Pin_2)
- new net RST: J7.3, U4.1 (~{RST})
- new net SCLK: U4.14 (SCLK)
- new net VCC: C4.1, J7.2, J8.5, P3.2, P4.2, U4.8 (VCC), U5.2 (VO)
- no-connect marks 0 -> 18
Other:
- note added: "CONNECTOR FOR P10 LED PANEL"
- note added: "CONNECTOR FOR PROGRAMMING"
- note added: "ESP-12Ex"
- note added: "JUMPER FOR PROGRAMMING"
- note added: "NUMBER CONTROLLER BUTTON"
- note added: "VOLTAGE REGULATOR FOR 3.3V"
- note removed: "10K"
- note removed: "10uf"
- note removed: "ESP-12EX"
- note removed: "GND"
- note removed: "Jumper"
- note removed: "RESET"
- note removed: "RX"
- note removed: "TX"
- note removed: "VCC"
- note removed: "VCC 3.3v"

Commit message: some small fixes
Connections:
- net GPIO2 is gone; now on net VCC: U4.17 (GPIO2)
- no-connect marks 18 -> 17
Changed lines of the file:
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@@
-	)
-	(no_connect
-		(at 128.27 55.88)
 	)
 	(no_connect
@@
 		)
 	)
-	(label "GPIO2"
-		(at 128.27 55.88 0)
-		(effects
-			(font
-				(size 1.27 1.27)
-			)
-			(justify left bottom)
-		)
-	)
 	(label "GPIO15"
 		(at 128.27 73.66 0)
@@
 		)
 	)
+	(label "VCC"
+		(at 128.27 55.88 0)
+		(effects
+			(font
+				(size 1.27 1.27)
+			)
+			(justify left bottom)
+		)
+		(property "VCC" ""
+			(at 128.27 55.88 0)
+			(effects
+				(font
+					(size 1.27 1.27)
+					(italic yes)
+				)
+			)
+		)
+	)

Commit message: added changes
Parts:
- J8: footprint MyConnectors:PinHeader_1x05_P2.54mm_Vertical -> Connector_PinHeader_2.54mm:PinHeader_1x02_P2.54mm_Vertical; symbol PCM_SL_Pin_Headers:PINHD_1x5_Male -> Connector_Generic:Conn_01x02
Connections:
- net EN: no longer J8.4
- net GND: now also J8.1 (Pin_1), U4.16 (GPIO15); no longer J8.3
- net GPIO0: now also J8.2 (Pin_2); no longer J8.1
- net GPIO15: no longer J8.2, U4.16 (GPIO15)
- net VCC: no longer J8.5
Changed lines of the file:
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@@
-		)
-	)
-	(label "EN"
-		(at 152.4 95.25 180)
-		(effects
-			(font
-				(size 1.27 1.27)
-			)
-			(justify right bottom)
-		)
-		(property "EN" ""
-			(at 152.4 95.25 0)
-			(effects
-				(font
-					(size 1.27 1.27)
-					(italic yes)
-				)
-			)
 		)
 	)
@@
 		)
 	)
-	(label "GPIO15"
-		(at 152.4 90.17 180)
-		(effects
-			(font
-				(size 1.27 1.27)
-			)
-			(justify right bottom)
-		)
-		(property "GPIO15" ""
-			(at 152.4 90.17 0)
-			(effects
-				(font
-					(size 1.27 1.27)
-					(italic yes)
-				)
-			)
-		)
-	)
 	(label "RST"
 		(at 97.79 50.8 180)
@@
 	)
 	(label "GPIO0"
-		(at 152.4 87.63 180)
+		(at 149.86 97.79 180)
 		(effects
 			(font
@@
 		)
 		(property "GPIO0" ""
-			(at 152.4 87.63 0)
+			(at 149.86 97.79 0)
 			(effects
 				(font
@@
 	)
 	(label "GND"
-		(at 152.4 92.71 180)
+		(at 149.86 95.25 180)
 		(effects
 			(font
@@
 		)
 		(property "GND" ""
-			(at 152.4 92.71 0)
+			(at 149.86 95.25 0)
 			(effects
 				(font
@@
 		)
 	)
-	(label "GPIO15"
+	(label "GND"
 		(at 128.27 73.66 0)
-		(effects
-			(font
-				(size 1.27 1.27)
-			)
-			(justify left bottom)
+		(fields_autoplaced yes)
+		(effects
+			(font
+				(size 1.27 1.27)
+			)
+			(justify left bottom)
+		)
+		(property "GND" ""
+			(at 128.27 74.93 0)
+			(effects
+				(font
+					(size 1.27 1.27)
+					(italic yes)
+				)
+				(justify left)
+			)
 		)
 	)
@@
 	)
 	(label "VCC"
-		(at 152.4 97.79 180)
-		(effects
-			(font
-				(size 1.27 1.27)
-			)
-			(justify right bottom)
-		)
-		(property "VCC" ""
-			(at 152.4 97.79 0)
-			(effects
-				(font
-					(size 1.27 1.27)
-					(italic yes)
-				)
-			)
-		)
-	)
-	(label "VCC"
 		(at 113.03 45.72 90)
 		(effects
@@
 	)
 	(symbol
-		(lib_id "PCM_SL_Pin_Headers:PINHD_1x5_Male")
-		(at 156.21 92.71 0)
+		(lib_id "Connector_Generic:Conn_01x02")
+		(at 154.94 95.25 0)
 		(unit 1)
 		(exclude_from_sim no)
@@
 		(fields_autoplaced yes)
 		(property "Reference" "J8"
-			(at 158.75 92.7099 0)
+			(at 157.48 96.5199 0)
 			(effects
 				(font
@@
 		)
 		(property "Value" "PINHD_1x5_Male"
-			(at 158.75 93.9799 0)
+			(at 157.48 96.5199 0)
 			(effects
 				(font
@@
 			)
 		)
-		(property "Footprint" "MyConnectors:PinHeader_1x05_P2.54mm_Vertical"
-			(at 154.94 80.01 0)
-			(effects
-				(font
-					(size 1.27 1.27)
-				)
-			)
-		)
-		(property "Datasheet" ""
-			(at 156.21 81.28 0)
+		(property "Footprint" "Connector_PinHeader_2.54mm:PinHeader_1x02_P2.54mm_Vertical"
+			(at 154.94 95.25 0)
 			(effects
 				(font
@@
 			)
 		)
-		(property "Description" "Pin Header male with pin space 2.54mm. Pin Count -5"
-			(at 156.21 92.71 0)
+		(property "Datasheet" "~"
+			(at 154.94 95.25 0)
 			(effects
 				(font
@@
 			)
 		)
+		(property "Description" "Generic connector, single row, 01x02, script generated (kicad-library-utils/schlib/autogen/connector/)"
+			(at 154.94 95.25 0)
+			(effects
+				(font
+					(size 1.27 1.27)
+				)
+				(hide yes)
+			)
+		)
 		(pin "1"
 		)
-		(pin "3"
-		)
-		(pin "5"
-		)
 		(pin "2"
 		)
-		(pin "4"
-		)
 		(instances

Commit message: fixed all errors
Connections:
- net EN is gone; now on net VCC: U4.3 (EN)
Changed lines of the file:
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@@
 		)
 	)
-	(label "EN"
+	(label "VCC"
 		(at 97.79 55.88 180)
+		(fields_autoplaced yes)
 		(effects
 			(font
@@
 			(justify right bottom)
 		)
+		(property "VCC" ""
+			(at 97.79 57.15 0)
+			(effects
+				(font
+					(size 1.27 1.27)
+					(italic yes)
+				)
+				(justify right)
+			)
+		)
 	)

Commit message: marked as final
Parts:
- renumbered C4 to C1, C3 to C2, J8 to J1, J7 to J2, J6 to J3, P3 to P1, P4 to P2, R3 to R1, R4 to R2, U4 to U1, U5 to U2
Other:
- note added: "1"
- note added: "2025-04-25"
- note added: "FINAL"
- note added: "P10 Lead Panel Controller using ESP-12E (ESP8266)"
- note added: "P10 Led Controller with ESP-12E, 12Ex"
- note added: "This board controlls the P10 Led board. Intended to use in Qeue Management System but can also be used in other sinage board display."
- moved on the sheet: C1, C2, J1, J2, J3, P1, P2, R1, R2, U1, U2
